File: Kicad/ATTiny3216.kicad_pcb (KiCad board)
At the start: 2 copper layers, 36.2 x 39.4 mm, 10 parts, among them J1 CONN_08SMD-STRAIGHT-FEMALE, J2 CONN_03SMD_RA_FEMALE, J3 CONN_08SMD-STRAIGHT-FEMALE, M1 LEDFAB1206, M2 FTDI-SMD-HEADER, U1 ATtiny3216

Commit message: Add files via upload
Other:
- net class Default removed
